File: afuue_project/KiCad/windsynth5_ver1.5/windsynyh5.sch (KiCad schematic (older format))
At the start: 35 parts, among them P1 SENSOR, P2 SPEAKER, P3 HEADPHONE, P4 EXT-POWER, P5 EXT, P6 AE-PAM8012, P7 I2C, P8 MIDI-TRS, U1 ESP32-DEVKIT-C, U2 TDA1543, U3 TDA1543

Commit message: AFUUE page の改善、MakerFaireTokyo2020向けのポップ、次期基板への準備など
Parts:
- R2, R3: value R -> 47
Connections:
- net at D1.2 (A), D3.2 (A): now also U1.8 (IO33); no longer U1.17 (SD3)
Changed lines of the file:
@@
 NoConn ~ 4900 2650
 NoConn ~ 4900 2750
-NoConn ~ 4900 3150
 NoConn ~ 4900 3950
 NoConn ~ 6000 3950
@@
 P 5900 6150
 F 0 "R3" V 5980 6150 50  0000 C CNN
-F 1 "R" V 5900 6150 50  0000 C CNN
+F 1 "47" V 5900 6150 50  0000 C CNN
 F 2 "Pin_Headers:Pin_Header_Straight_1x02_Pitch2.54mm" V 5830 6150 50  0001 C CNN
 F 3 "" H 5900 6150 50  0000 C CNN
@@
 P 5900 5950
 F 0 "R2" V 5980 5950 50  0000 C CNN
-F 1 "R" V 5900 5950 50  0000 C CNN
+F 1 "47" V 5900 5950 50  0000 C CNN
 F 2 "Pin_Headers:Pin_Header_Straight_1x02_Pitch2.54mm" V 5830 5950 50  0001 C CNN
 F 3 "" H 5900 5950 50  0000 C CNN
@@
 	6400 2850 6400 5150
 Wire Wire Line
-	6400 5150 8300 5150
-Wire Wire Line
 	6000 2550 6300 2550
 Wire Wire Line
@@
 	6150 5500 5850 5500
 Wire Wire Line
-	4900 4050 4450 4050
-Wire Wire Line
-	4450 4050 4450 5550
+	4450 3150 4450 5550
 $Comp
 L +3.3V #PWR05
@@
 Wire Wire Line
 	3450 4000 3100 4000
+Wire Wire Line
+	6400 5150 8300 5150
+Wire Wire Line
+	4900 3150 4450 3150
+NoConn ~ 4900 4050
 $EndSCHEMATC

Commit message: 現状のものを一旦コミット（KORG NTS-1対応含む）
Parts:
- removed GS1, GS2: GS, Connectors:GS2, symbol GS2
- removed U2: TDA1543, Housings_SOIC:SO-8_5.3x6.2mm_Pitch1.27mm, symbol TDA1543
- removed U3: TDA1543, Housings_DIP:DIP-8_W7.62mm, symbol TDA1543
- added C1: C, Pin_Headers:Pin_Header_Straight_1x02_Pitch2.54mm, symbol C
- P5: footprint Pin_Headers:Pin_Header_Straight_1x04_Pitch2.54mm -> Socket_Strips:Socket_Strip_Angled_1x04_Pitch2.54mm
- P8: value MIDI-TRS -> TRS MIDI
Connections:
- net +3V3 is gone; now on an unnamed net: D5.2 (A), P1.1 (P1), P7.2 (P2), R2.1, U1.1 (3V3)
- net GND: now also C1.2
- net at P4.2 (P2): no longer U1.18 (CMD)
- net at U1.25 (IO0): no longer P5.2 (P2)
- net at U1.26 (IO4): now also KeyUP1.1; no longer P5.3 (P3)
- net at U1.34 (RXD0): no longer KeyUP1.1
- net at U1.7 (IO32): now also P5.2 (P2)
- net at D1.2 (A), D3.2 (A), U1.8 (IO33): now also P5.3 (P3)
- net at U1.9 (IO25): now also R1.1
- net at R1.2, RV1.3: now also C1.1
- no-connect marks 18 -> 19
Other:
- note added: "Modified : RXD0 -> IO4"
- moved on the sheet: R1

Commit message: 基板発注したので
Parts:
- removed D1, D3, D5: D, Pin_Headers:Pin_Header_Straight_1x02_Pitch2.54mm, symbol D
- removed D4, D6: Led_Small, Pin_Headers:Pin_Header_Straight_1x02_Pitch2.54mm, symbol Led_Small
- P1: footprint Socket_Strips:Socket_Strip_Angled_1x04_Pitch2.54mm -> Socket_Strips:Socket_Strip_Angled_1x04_Pitch2.00mm
- P2: footprint Pin_Headers:Pin_Header_Straight_1x02_Pitch2.54mm -> UGSM30:USGM30
- P4: footprint Socket_Strips:Socket_Strip_Straight_1x03_Pitch2.54mm -> Socket_Strips:Socket_Strip_Straight_1x03_Pitch2.00mm
- P7: footprint Pin_Headers:Pin_Header_Straight_1x05_Pitch2.54mm -> Pin_Headers:Pin_Header_Straight_1x05_Pitch2.00mm
- renumbered D2 to D1
Connections:
- net at P5.3 (P3), U1.8 (IO33): now also D1.2 (A)
Changed lines of the file:
@@
 F 0 "P1" H 6650 1300 50  0000 C CNN
 F 1 "SENSOR" V 6750 1050 50  0000 C CNN
-F 2 "Socket_Strips:Socket_Strip_Angled_1x04_Pitch2.54mm" H 6650 1050 50  0001 C CNN
+F 2 "Socket_Strips:Socket_Strip_Angled_1x04_Pitch2.00mm" H 6650 1050 50  0001 C CNN
 F 3 "" H 6650 1050 50  0000 C CNN
 	1    6650 1050
@@
 F 0 "P2" H 3250 2000 50  0000 C CNN
 F 1 "SPEAKER" V 3350 1850 50  0000 C CNN
-F 2 "Pin_Headers:Pin_Header_Straight_1x02_Pitch2.54mm" H 3250 1850 50  0001 C CNN
+F 2 "UGSM30:USGM30" H 3250 1850 50  0001 C CNN
 F 3 "" H 3250 1850 50  0000 C CNN
 	1    3250 1850
@@
 F 0 "P7" H 5750 1350 50  0000 C CNN
 F 1 "I2C" V 5850 1050 50  0000 C CNN
-F 2 "Pin_Headers:Pin_Header_Straight_1x05_Pitch2.54mm" H 5750 1050 50  0001 C CNN
+F 2 "Pin_Headers:Pin_Header_Straight_1x05_Pitch2.00mm" H 5750 1050 50  0001 C CNN
 F 3 "" H 5750 1050 50  0000 C CNN
 	1    5750 1050
@@
 $EndComp
 $Comp
-L Led_Small D2
+L Led_Small D1
 U 1 1 5F3D4A68
 P 3700 5150
-F 0 "D2" H 3650 5275 50  0000 L CNN
+F 0 "D1" H 3650 5275 50  0000 L CNN
 F 1 "Led_Small" H 3525 5050 50  0000 L CNN
 F 2 "Pin_Headers:Pin_Header_Straight_1x02_Pitch2.54mm" V 3700 5150 50  0001 C CNN
@@
 	1    0    0    -1
 $EndComp
-$Comp
-L Led_Small D4
-U 1 1 5F3D4B28
-P 3700 5550
-F 0 "D4" H 3650 5675 50  0000 L CNN
-F 1 "Led_Small" H 3525 5450 50  0000 L CNN
-F 2 "Pin_Headers:Pin_Header_Straight_1x02_Pitch2.54mm" V 3700 5550 50  0001 C CNN
-F 3 "" V 3700 5550 50  0000 C CNN
-	1    3700 5550
-	1    0    0    -1
-$EndComp
-$Comp
-L D D1
-U 1 1 5F3E8C46
-P 4150 5150
-F 0 "D1" H 4150 5250 50  0000 C CNN
-F 1 "D" H 4150 5050 50  0000 C CNN
-F 2 "Pin_Headers:Pin_Header_Straight_1x02_Pitch2.54mm" H 4150 5150 50  0001 C CNN
-F 3 "" H 4150 5150 50  0000 C CNN
-	1    4150 5150
-	1    0    0    -1
-$EndComp
-$Comp
-L D D3
-U 1 1 5F3E8CC2
-P 4150 5550
-F 0 "D3" H 4150 5650 50  0000 C CNN
-F 1 "D" H 4150 5450 50  0000 C CNN
-F 2 "Pin_Headers:Pin_Header_Straight_1x02_Pitch2.54mm" H 4150 5550 50  0001 C CNN
-F 3 "" H 4150 5550 50  0000 C CNN
-	1    4150 5550
-	1    0    0    -1
-$EndComp
 Wire Wire Line
 	6000 3550 6900 3550
@@
 Wire Wire Line
 	3600 5150 3500 5150
-Wire Wire Line
-	3500 4850 3500 5900
 Connection ~ 3500 4850
 Wire Wire Line
-	3500 5550 3600 5550
-Connection ~ 3500 5150
-Wire Wire Line
-	3800 5550 4000 5550
-Wire Wire Line
-	3800 5150 4000 5150
-Wire Wire Line
-	4450 5150 4300 5150
-Wire Wire Line
-	4300 5550 5500 5550
+	3800 5150 4450 5150
+Wire Wire Line
+	4450 5550 5500 5550
 Connection ~ 4450 5150
-$Comp
-L Led_Small D6
-U 1 1 5F478FDD
-P 3700 5900
-F 0 "D6" H 3650 6025 50  0000 L CNN
-F 1 "Led_Small" H 3525 5800 50  0000 L CNN
-F 2 "Pin_Headers:Pin_Header_Straight_1x02_Pitch2.54mm" V 3700 5900 50  0001 C CNN
-F 3 "" V 3700 5900 50  0000 C CNN
-	1    3700 5900
-	1    0    0    -1
-$EndComp
-$Comp
-L D D5
-U 1 1 5F479067
-P 4150 5900
-F 0 "D5" H 4150 6000 50  0000 C CNN
-F 1 "D" H 4150 5800 50  0000 C CNN
-F 2 "Pin_Headers:Pin_Header_Straight_1x02_Pitch2.54mm" H 4150 5900 50  0001 C CNN
-F 3 "" H 4150 5900 50  0000 C CNN
-	1    4150 5900
-	1    0    0    -1
-$EndComp
-Wire Wire Line
-	4800 5900 4300 5900
-Connection ~ 4800 5900
-Wire Wire Line
-	4000 5900 3800 5900
-Wire Wire Line
-	3500 5900 3600 5900
-Connection ~ 3500 5550
 Wire Wire Line
 	6000 3650 6400 3650
@@
 F 0 "P4" H 2900 4200 50  0000 C CNN
 F 1 "EXT-POWER" V 3000 4000 50  0000 C CNN
-F 2 "Socket_Strips:Socket_Strip_Straight_1x03_Pitch2.54mm" H 2900 4000 50  0001 C CNN
+F 2 "Socket_Strips:Socket_Strip_Straight_1x03_Pitch2.00mm" H 2900 4000 50  0001 C CNN
 F 3 "" H 2900 4000 50  0000 C CNN
 	1    2900 4000
@@
 Wire Wire Line
 	5500 5750 5500 5550
-Connection ~ 4450 5550
 NoConn ~ 6000 2850
 Wire Wire Line
@@
 	3350 3650 2750 3650
 Connection ~ 2750 3650
+Wire Wire Line
+	3500 5150 3500 4850
 $EndSCHEMATC
