File: afuue_project/KiCad/windsynth5_ver1.6/windsynyh5.kicad_pcb (KiCad board)
At the start: 2 copper layers, 74.9 x 125.7 mm, 30 parts, among them SW1 SW_SPDT

Commit message: v6向け更新
Parts:
- moved SW1 2.54 mm to (180.3, 172.1)
- moved VOLUME 2.35 mm to (179.7, 160.8)
- renumbered KeyUp to KeyUP
Connections:
- ESP32-DEVKIT-C (*) pad 35: Net-(R2-Pad1) -> Net-(R3-Pad1)
- R2 pad 1: Net-(R2-Pad1) -> Net-(P1-Pad2)
- R3 pad 1: Net-(P1-Pad2) -> Net-(R3-Pad1)
Routing:
- net Net-(R2-Pad1): track 35.9 -> 0.00 mm
- net Net-(R3-Pad1): track 0.00 -> 35.2 mm
- net Net-(P3-Pad2): track 90.0 -> 98.2 mm
- net Net-(P1-Pad2): track 139.6 -> 143.9 mm
- net Net-(P3-Pad3): track 125.3 -> 127.7 mm
- net GND: track 477.0 -> 478.4 mm
- net Net-(P4-Pad1): track 62.4 -> 63.6 mm
- net +9V: track 37.3 -> 36.4 mm
- net Net-(C1-Pad1): track 18.8 -> 18.0 mm
Other:
- board text added: "AFUUE BOARD VER1.6C - 21/04/09 @OtooneDev"
- board text removed: "AFUUE BOARD VER1.6B - 21/02/14 @OtooneDev"
