File: afuue_project/KiCad/windsynth9/face/face/face.kicad_pcb (KiCad board)
At the start: 2 copper layers, 132 x 64 mm, 5 parts, among them J1 Conn_01x02_Female, J2 Conn_01x02_Female

Commit message: AFUUE2 PWMx2 Version (1.9c)
Routing:
- net GND: vias 6 -> 4
Other:
- outline, holes or cut-outs redrawn
- board text added: "JLCJLCJLCJLC"
Changed lines of the file:
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@@
   (general
     (thickness 1.6)
-    (drawings 69)
-    (tracks 50)
+    (drawings 72)
+    (tracks 48)
     (zones 0)
     (modules 5)
@@
       ))
   )
+  (gr_text JLCJLCJLCJLC (at 89 128) (layer B.Adhes)
+    (effects (font (size 1 1) (thickness 0.15)) (justify mirror))
+  )
+  (gr_line (start 104 77) (end 101.894427 71.552786) (layer Edge.Cuts) (width 0.05))
+  (dimension 3 (width 0.15) (layer Dwgs.User)
+    (gr_text "3.000 mm" (at 102.5 67.2) (layer Dwgs.User)
+      (effects (font (size 1 1) (thickness 0.15)))
+    )
+    (feature1 (pts (xy 101 71) (xy 101 67.913579)))
+    (feature2 (pts (xy 104 71) (xy 104 67.913579)))
+    (crossbar (pts (xy 104 68.5) (xy 101 68.5)))
+    (arrow1a (pts (xy 101 68.5) (xy 102.126504 67.913579)))
+    (arrow1b (pts (xy 101 68.5) (xy 102.126504 69.086421)))
+    (arrow2a (pts (xy 104 68.5) (xy 102.873496 67.913579)))
+    (arrow2b (pts (xy 104 68.5) (xy 102.873496 69.086421)))
+  )
+  (dimension 5 (width 0.15) (layer Dwgs.User)
+    (gr_text "5.000 mm" (at 107.3 74.5 270) (layer Dwgs.User)
+      (effects (font (size 1 1) (thickness 0.15)))
+    )
+    (feature1 (pts (xy 104 77) (xy 106.586421 77)))
+    (feature2 (pts (xy 104 72) (xy 106.586421 72)))
+    (crossbar (pts (xy 106 72) (xy 106 77)))
+    (arrow1a (pts (xy 106 77) (xy 105.413579 75.873496)))
+    (arrow1b (pts (xy 106 77) (xy 106.586421 75.873496)))
+    (arrow2a (pts (xy 106 72) (xy 105.413579 73.126504)))
+    (arrow2b (pts (xy 106 72) (xy 106.586421 73.126504)))
+  )
+  (gr_line (start 104 129) (end 101.894427 134.447214) (layer Edge.Cuts) (width 0.05))
+  (dimension 3 (width 0.15) (layer Dwgs.User)
+    (gr_text "3.000 mm" (at 102.5 138.3) (layer Dwgs.User)
+      (effects (font (size 1 1) (thickness 0.15)))
+    )
+    (feature1 (pts (xy 101 135) (xy 101 137.586421)))
+    (feature2 (pts (xy 104 135) (xy 104 137.586421)))
+    (crossbar (pts (xy 104 137) (xy 101 137)))
+    (arrow1a (pts (xy 101 137) (xy 102.126504 136.413579)))
+    (arrow1b (pts (xy 101 137) (xy 102.126504 137.586421)))
+    (arrow2a (pts (xy 104 137) (xy 102.873496 136.413579)))
+    (arrow2b (pts (xy 104 137) (xy 102.873496 137.586421)))
+  )
+  (dimension 5 (width 0.15) (layer Dwgs.User)
+    (gr_text "5.000 mm" (at 108.3 131.5 90) (layer Dwgs.User)
+      (effects (font (size 1 1) (thickness 0.15)))
+    )
+    (feature1 (pts (xy 104 129) (xy 107.586421 129)))
+    (feature2 (pts (xy 104 134) (xy 107.586421 134)))
+    (crossbar (pts (xy 107 134) (xy 107 129)))
+    (arrow1a (pts (xy 107 129) (xy 107.586421 130.126504)))
+    (arrow1b (pts (xy 107 129) (xy 106.413579 130.126504)))
+    (arrow2a (pts (xy 107 134) (xy 107.586421 132.873496)))
+    (arrow2b (pts (xy 107 134) (xy 106.413579 132.873496)))
+  )
   (dimension 20.5 (width 0.15) (layer Dwgs.User)
     (gr_text "20.500 mm" (at 196.75 146.8) (layer Dwgs.User)
@@
     (arrow2b (pts (xy 94 83) (xy 95.126504 82.413579)))
   )
-  (dimension 8.5 (width 0.15) (layer Dwgs.User)
-    (gr_text "8.500 mm" (at 205.8 112.75 90) (layer Dwgs.User)
-      (effects (font (size 1 1) (thickness 0.15)))
-    )
-    (feature1 (pts (xy 194 108.5) (xy 205.086421 108.5)))
-    (feature2 (pts (xy 194 117) (xy 205.086421 117)))
-    (crossbar (pts (xy 204.5 117) (xy 204.5 108.5)))
-    (arrow1a (pts (xy 204.5 108.5) (xy 205.086421 109.626504)))
-    (arrow1b (pts (xy 204.5 108.5) (xy 203.913579 109.626504)))
-    (arrow2a (pts (xy 204.5 117) (xy 205.086421 115.873496)))
-    (arrow2b (pts (xy 204.5 117) (xy 203.913579 115.873496)))
-  )
-  (dimension 8.5 (width 0.15) (layer Dwgs.User)
-    (gr_text "8.500 mm" (at 205.8 93.25 270) (layer Dwgs.User)
-      (effects (font (size 1 1) (thickness 0.15)))
-    )
-    (feature1 (pts (xy 194 97.5) (xy 205.086421 97.5)))
-    (feature2 (pts (xy 194 89) (xy 205.086421 89)))
-    (crossbar (pts (xy 204.5 89) (xy 204.5 97.5)))
-    (arrow1a (pts (xy 204.5 97.5) (xy 203.913579 96.373496)))
-    (arrow1b (pts (xy 204.5 97.5) (xy 205.086421 96.373496)))
-    (arrow2a (pts (xy 204.5 89) (xy 203.913579 90.126504)))
-    (arrow2b (pts (xy 204.5 89) (xy 205.086421 90.126504)))
-  )
   (dimension 4.5 (width 0.15) (layer Dwgs.User)
     (gr_text "4.500 mm" (at 199.75 81.7) (layer Dwgs.User)
@@
     (arrow2a (pts (xy 75 62.5) (xy 76.126504 63.086421)))
     (arrow2b (pts (xy 75 62.5) (xy 76.126504 61.913579)))
-  )
-  (dimension 16 (width 0.15) (layer Dwgs.User)
-    (gr_text "16.000 mm" (at 219.3 103 90) (layer Dwgs.User)
-      (effects (font (size 1 1) (thickness 0.15)))
-    )
-    (feature1 (pts (xy 186.5 95) (xy 218.586421 95)))
-    (feature2 (pts (xy 186.5 111) (xy 218.586421 111)))
-    (crossbar (pts (xy 218 111) (xy 218 95)))
-    (arrow1a (pts (xy 218 95) (xy 218.586421 96.126504)))
-    (arrow1b (pts (xy 218 95) (xy 217.413579 96.126504)))
-    (arrow2a (pts (xy 218 111) (xy 218.586421 109.873496)))
-    (arrow2b (pts (xy 218 111) (xy 217.413579 109.873496)))
-  )
-  (dimension 24 (width 0.15) (layer Dwgs.User)
-    (gr_text "24.000 mm" (at 179.7 123 90) (layer Dwgs.User)
-      (effects (font (size 1 1) (thickness 0.15)))
-    )
-    (feature1 (pts (xy 198 111) (xy 180.413579 111)))
-    (feature2 (pts (xy 198 135) (xy 180.413579 135)))
-    (crossbar (pts (xy 181 135) (xy 181 111)))
-    (arrow1a (pts (xy 181 111) (xy 181.586421 112.126504)))
-    (arrow1b (pts (xy 181 111) (xy 180.413579 112.126504)))
-    (arrow2a (pts (xy 181 135) (xy 181.586421 133.873496)))
-    (arrow2b (pts (xy 181 135) (xy 180.413579 133.873496)))
   )
   (dimension 15.5 (width 0.15) (layer Dwgs.User)
@@
     (arrow2b (pts (xy 130 71) (xy 130.586421 72.126504)))
   )
-  (gr_line (start 104 72) (end 104 88) (layer Edge.Cuts) (width 0.05))
+  (gr_line (start 104 77) (end 104 88) (layer Edge.Cuts) (width 0.05))
   (gr_line (start 198 72) (end 198 88) (layer Edge.Cuts) (width 0.05))
   (dimension 18 (width 0.15) (layer Dwgs.User)
@@
   (gr_arc (start 199 72) (end 199 71) (angle -90) (layer Edge.Cuts) (width 0.05))
   (gr_line (start 105 89) (end 197 89) (layer Edge.Cuts) (width 0.05))
-  (gr_arc (start 103 72) (end 104 72) (angle -90) (layer Edge.Cuts) (width 0.05))
-  (gr_line (start 103 71) (end 81 71) (layer Edge.Cuts) (width 0.05))
+  (gr_arc (start 101 72) (end 101 71) (angle 63.43494882) (layer Edge.Cuts) (width 0.05))
+  (gr_line (start 101 71) (end 81 71) (layer Edge.Cuts) (width 0.05))
   (gr_line (start 199 135) (end 201 135) (layer Edge.Cuts) (width 0.05))
   (gr_arc (start 201 129) (end 201 135) (angle -90) (layer Edge.Cuts) (width 0.05))
@@
   (gr_line (start 198 118) (end 198 134) (layer Edge.Cuts) (width 0.05))
   (gr_line (start 105 117) (end 197 117) (layer Edge.Cuts) (width 0.05))
-  (gr_line (start 104 134) (end 104 118) (layer Edge.Cuts) (width 0.05))
-  (gr_arc (start 103 134) (end 103 135) (angle -90) (layer Edge.Cuts) (width 0.05))
-  (gr_line (start 81 135) (end 103 135) (layer Edge.Cuts) (width 0.05))
+  (gr_line (start 104 129) (end 104 118) (layer Edge.Cuts) (width 0.05))
+  (gr_arc (start 101 134) (end 101 135) (angle -63.43494882) (layer Edge.Cuts) (width 0.05))
+  (gr_line (start 81 135) (end 101 135) (layer Edge.Cuts) (width 0.05))
   (dimension 18 (width 0.15) (layer Dwgs.User)
     (gr_text "18.000 mm" (at 215.8 126 90) (layer Dwgs.User)
@@
   (segment (start 82 122.5) (end 83 121.5) (width 0.25) (layer B.Cu) (net 2))
   (segment (start 82 128) (end 82 122.5) (width 0.25) (layer B.Cu) (net 2))
-  (via (at 186.5 111) (size 3.4) (drill 3.2) (layers F.Cu B.Cu) (net 2))
-  (via (at 186.5 95) (size 3.4) (drill 3.2) (layers F.Cu B.Cu) (net 2))
   (zone (net 2) (net_name GND) (layer B.Cu) (hatch edge 0.508)
     (connect_pads (clearance 0.508))
