File: afuue_project/KiCad/windsynth9/windsynth/windsynth.kicad_pcb (KiCad board)
At the start: 2 copper layers, 117 x 64 mm, 38 parts, among them J7 Conn_01x02, M5StickC M5StickC

Commit message: AFUUE2 PWMx2 Version (1.9c)
Parts:
- removed EXTRA: ExtraPort, Connector_PinHeader_2.54mm:PinHeader_1x02_P2.54mm_Vertical
- removed G***: , Logo:otoonedev_logo
- removed I2C: I2C, Connector_PinHeader_2.00mm:PinHeader_1x04_P2.00mm_Horizontal
- removed I2C: ExtraI2C, Connector_PinHeader_2.00mm:PinHeader_1x04_P2.00mm_Vertical
- removed PCF8574 (x2): PCF8574, Package_SO:SOIC-16W_7.5x12.8mm_P1.27mm
- added ADC-DIRECT: Conn_01x02, Jumper:SolderJumper-2_P1.3mm_Open_RoundedPad1.0x1.5mm, F.Cu at (156.5, 94.0)
- added C2: CP_Small, Connector_PinHeader_2.54mm:PinHeader_1x02_P2.54mm_Vertical, B.Cu at (127.0, 115.5)
- added J1: I2C, Connector_JST:JST_PH_B4B-PH-SM4-TB_1x04-1MP_P2.00mm_Vertical, F.Cu at (215.0, 92.0)
- added J10: BleathSensor, DIP6_Reverse:DIP-6_W7.62mm_Reverse, F.Cu at (171.5, 100.0)
- added J2: ExtraI2C, Connector_PinHeader_2.00mm:PinHeader_1x04_P2.00mm_Vertical, F.Cu at (229.0, 89.0)
- added R2: R, Connector_PinHeader_2.54mm:PinHeader_1x02_P2.54mm_Vertical, F.Cu at (178.0, 106.0)
- added U1: MCP3425A0T-ECH, Package_TO_SOT_SMD:SOT-23-6_Handsoldering, F.Cu at (197.0, 97.5)
- added U2: MCP3425A0T-ECH, Package_TO_SOT_SMD:SOT-23-6_Handsoldering, F.Cu at (206.5, 97.5)
- C1: value C_Small -> CP; moved to B.Cu
- J7: footprint Connector_PinHeader_2.54mm:PinHeader_1x02_P2.54mm_Vertical -> Jumper:SolderJumper-2_P1.3mm_Open_RoundedPad1.0x1.5mm; moved to B.Cu
- R1: value 510 -> R
- moved C1 8.50 mm to (161.0, 96.0), turned to 270 degrees
- moved R1 8.14 mm to (169.0, 106.0), turned to 270 degrees
- moved J7 7.80 mm to (181.5, 106.0), turned to 0 degrees
- moved J9 2.00 mm to (153.0, 100.0)
- renumbered M5StickC to J3, AE-PAM8012 to J4, SPEAKER to J5, HEADPHONE to J8, MIS2503 to J9, VOLUME to RV1, KeyC to SW1, KeyB to SW10, KeyDown to SW11, KeyUp to SW12, KeyEb to SW2, KeyD to SW3, KeyE to SW4, KeyF to SW5, KeyCs to SW6, KeyGs to SW7, KeyG to SW8, KeyA to SW9, MCP23017 to U3
Connections:
- C1 pad 1: GND -> +3V3
- C1 pad 2: Net-(C1-Pad2) -> GND
- J3 pad 2: Net-(J3-Pad2) -> +5V
- J3 pad 4: Net-(J3-Pad3) -> Net-(J3-Pad4)
- J3 pad 7: Net-(J3-Pad7) -> +3V3
- J4 pad 1: Net-(J3-Pad2) -> +5V
- J8 pad 2: Net-(J8-Pad2) -> Net-(C2-Pad2)
- J8 pad 5: Net-(J8-Pad2) -> Net-(C2-Pad2)
- J9 pad 4: Net-(J3-Pad7) -> +3V3
- J9 pad 5: Net-(J3-Pad3) -> Net-(J6-Pad1)
- R1 pad 2: Net-(C1-Pad2) -> Net-(R1-Pad2)
- RV1 pad 2: Net-(J8-Pad2) -> Net-(C2-Pad1)
- RV1 pad 3: Net-(C1-Pad2) -> Net-(R1-Pad2)
- U3 pad 18: +5V -> +3V3
- U3 pad 9: +5V -> +3V3
Routing:
- net GND: track 460.2 -> 98.8 mm, vias 18 -> 5
- net +3V3: track 0.00 -> 129.3 mm, vias 0 -> 5
- net Net-(J6-Pad1): track 0.00 -> 60.0 mm, vias 0 -> 1
- net Net-(J8-Pad2): track 58.0 -> 0.00 mm
- net Net-(C2-Pad2): track 0.00 -> 57.3 mm
- net Net-(SW6-Pad1): track 101.2 -> 47.8 mm
- net Net-(J3-Pad2): track 51.8 -> 0.00 mm, vias 1 -> 0
- net Net-(R1-Pad2): track 0.00 -> 48.8 mm
- net Net-(C1-Pad2): track 45.1 -> 0.00 mm
- net Net-(J10-Pad5): track 0.00 -> 33.3 mm, vias 0 -> 2
- net Net-(J3-Pad7): track 30.0 -> 0.00 mm
- net Net-(J3-Pad3): track 47.3 -> 18.8 mm
- net Net-(J3-Pad4): track 0.00 -> 25.8 mm
- net Net-(SW5-Pad1): track 98.0 -> 73.6 mm
- net Net-(SW10-Pad1): track 84.3 -> 64.0 mm, vias 2 -> 0
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Other:
- board text added: "(Main)"
- board text added: "(Sub)"
- board text added: "+"
- board text added: "AFUUE BOARD Ver 1.9d 2023/07/08 @OtooneDev"
- board text removed: "AFUUE BOARD Ver 1.9b 2022/08/28 @OtooneDev"
