File: afuue_project/KiCad/windsynth9/windsynth/windsynth.sch (KiCad schematic (older format))
At the start: 37 parts, among them J1 I2C, J2 ExtraI2C, J3 M5StickC, J4 PAM8012, J5 SpeakerOut, J6 ExtraPort, J7 Conn_01x02, J8 StereoMiniJack, J9 BleathSensor, SW1 SW_with_LED, SW10 SW_with_LED, SW11 SW_with_LED, SW12 SW_with_LED, SW2 SW_with_LED, SW3 SW_with_LED, SW4 SW_with_LED, SW5 SW_with_LED, SW6 SW_with_LED, SW7 SW_with_LED, SW8 SW_with_LED, SW9 SW_with_LED, U1 PCF8574, U2 PCF8574, U3 MCP23017_SO

Commit message: AFUUE2 PWMx2 Version (1.9c)
Parts:
- removed C1: C_Small, Connector_PinHeader_2.54mm:PinHeader_1x02_P2.54mm_Vertical, symbol Device:C_Small
- removed U1, U2: PCF8574, Package_SO:SOIC-16W_7.5x12.8mm_P1.27mm, symbol Interface_Expansion:PCF8574
- added C1: CP, Connector_PinHeader_2.54mm:PinHeader_1x02_P2.54mm_Vertical, symbol Device:CP
- added C2: CP_Small, Connector_PinHeader_2.54mm:PinHeader_1x02_P2.54mm_Vertical, symbol Device:CP_Small
- added J10: BleathSensor, DIP6_Reverse:DIP-6_W7.62mm_Reverse, symbol Connector_Generic:Conn_02x03_Counter_Clockwise
- added R2: R, Connector_PinHeader_2.54mm:PinHeader_1x02_P2.54mm_Vertical, symbol Device:R
- added U1, U2: MCP3425A0T-ECH, Package_TO_SOT_SMD:SOT-23-6_Handsoldering, symbol Analog_ADC:MCP3425A0T-ECH
- J1: footprint Connector_PinHeader_2.00mm:PinHeader_1x04_P2.00mm_Horizontal -> Connector_JST:JST_PH_B4B-PH-SM4-TB_1x04-1MP_P2.00mm_Vertical
- J6: value ExtraPort -> Conn_01x02; footprint Connector_PinHeader_2.54mm:PinHeader_1x02_P2.54mm_Vertical -> Jumper:SolderJumper-2_P1.3mm_Open_RoundedPad1.0x1.5mm
- J7: footprint Connector_PinHeader_2.54mm:PinHeader_1x02_P2.54mm_Vertical -> Jumper:SolderJumper-2_P1.3mm_Open_RoundedPad1.0x1.5mm
- R1: value 510 -> R
Connections:
- net +5V: now also J3.2 (Pin_2), J4.1 (Pin_1); no longer J1.3 (Pin_3), J2.3 (Pin_3), U3.18 (~RESET~), U3.9 (VDD)
- net GND: now also C1.2, J10.6 (Pin_6), U1.2 (Vss), U1.6 (Vin-), U2.2 (Vss), U2.6 (Vin-); no longer J6.2 (Pin_2)
- net at J1.1 (Pin_1), J2.1 (Pin_1), U3.12 (SCK): now also U1.3 (SCL), U2.3 (SCL)
- net at J1.2 (Pin_2), J2.2 (Pin_2), U3.13 (SDA): now also U1.4 (SDA), U2.4 (SDA)
- net at J3.3 (Pin_3), R1.1: no longer J3.4 (Pin_4), J9.5 (Pin_5)
- net at J3.5 (Pin_5): now also R2.1; no longer J6.1 (Pin_1)
- net +3V3: now reaches J3.7 (Pin_7), J9.4 (Pin_4)
- net +3V3: now also J1.3 (Pin_3), J2.3 (Pin_3), U3.18 (~RESET~), U3.9 (VDD), C1.1, J10.4 (Pin_4), U1.5 (Vdd), U2.5 (Vdd)
- net at J8.2 (Pin_2), J8.5 (Pin_5): now also C2.2; no longer RV1.2
- net at R1.2, RV1.3: now also R2.2
- new net: J3.4 (Pin_4), J6.2 (Pin_2)
- new net: C2.1, RV1.2
- new net: J6.1 (Pin_1), J9.5 (Pin_5), U1.1 (Vin+)
- new net: J10.5 (Pin_5), U2.1 (Vin+)
- no-connect marks 23 -> 20
